Commit message: add robotiq visual

File: ur10e_robotiq_simplified_description/urdf/ur10e_robotiq.urdf.xacro (robot description, xacro)
@@ -6,4 +6,5 @@
   <!-- ur10e -->
   <xacro:include filename="$(find ur_simplified_description)/urdf/ur10e.urdf.xacro" />
+	<xacro:include filename="$(find ur10e_robotiq_simplified_description)/urdf/robotiq_arg2f_85_model_macro.xacro" />
   <!-- gripper -->
   <joint name="rq_coupler_joint" type="fixed">
@@ -23,7 +24,7 @@
   </visual>
   <collision>
-      <origin xyz="0 0 0.005" rpy="0 0 0" />
+      <origin xyz="0 0 0.02" rpy="0 0 0" />
        <geometry>
-        <cylinder radius="${0.075*0.5}" length="0.01"/>
+        <cylinder radius="${0.075*0.5}" length="0.04"/>
        </geometry>
        <material name="RobotiqGrey">
@@ -36,4 +37,10 @@
   </inertial>
   </link>
+    <joint name="robotiq_joint" type="fixed">
+    <parent link="robotiq_coupler" />
+    <child link = "robotiq_arg2f_base_link" />
+    <origin xyz="0.0 0.0 0.0" rpy="0 0 ${0.0*pi}" />
+  </joint>
+    <xacro:robotiq_arg2f_85 prefix=""/>
   <link name="robotiq_simplified">
     <inertial>
@@ -42,13 +49,4 @@
       <inertia ixx="0.00020005" ixy="-4.2442E-10" ixz="-2.9069E-10" iyy="0.00017832" iyz="-3.4402E-08" izz="0.00013478" />
     </inertial>
-    <visual>
-      <origin xyz="0 0 0.075" rpy="0 0 0" />
-      <geometry>
-        <box size="0.035 0.145 0.15"/>
-      </geometry>
-      <material name="">
-        <color rgba="0.1 0.1 0.1 1" />
-      </material>
-    </visual>
     <collision>
       <origin xyz="0 0 0.075" rpy="0 0 0" />
@@ -56,7 +54,10 @@
          <box size="0.035 0.145 0.15"/>
       </geometry>
+             <material name="RobotiqGrey">
+         <color rgba="0.1 0.1 0.1 1"/>
+       </material>
     </collision>
   </link>
-      <joint name="robotiq_joint" type="fixed">
+      <joint name="robotiq_joint_simplified" type="fixed">
       <parent link="robotiq_coupler" />
       <child link = "robotiq_simplified" />
@@ -84,5 +85,5 @@
        <origin xyz="0 0 0" rpy="0 0 0" />
        <geometry>
-         <box size="0.04 0.04 0.04" />
+         <box size="0.02 0.02 0.04" />
        </geometry>
        <material name="White">
@@ -93,5 +94,5 @@
      <origin xyz="0 0 0" rpy="0 0 0" />
      <geometry>
-       <box size="0.04 0.04 0.04" />
+       <box size="0.02 0.02 0.04" />
      </geometry>
      <material name="White">

Commit message: improved collision shape gripper

File: ur10e_robotiq_simplified_description/urdf/ur10e_robotiq.urdf.xacro (robot description, xacro)
@@ -50,7 +50,25 @@
     </inertial>
     <collision>
-      <origin xyz="0 0 0.075" rpy="0 0 0" />
+      <origin xyz="0 0 0.045" rpy="0 0 0" />
       <geometry>
-         <box size="0.035 0.145 0.15"/>
+         <box size="0.035 0.145 0.09"/>
+      </geometry>
+             <material name="RobotiqGrey">
+         <color rgba="0.1 0.1 0.1 1"/>
+       </material>
+    </collision>
+    <collision>
+      <origin xyz="0 0.055 0.08" rpy="0 0 0" />
+      <geometry>
+         <box size="0.035 0.03 0.16"/>
+      </geometry>
+             <material name="RobotiqGrey">
+         <color rgba="0.1 0.1 0.1 1"/>
+       </material>
+    </collision>
+    <collision>
+      <origin xyz="0 -0.055 0.08" rpy="0 0 0" />
+      <geometry>
+         <box size="0.035 0.03 0.16"/>
       </geometry>
              <material name="RobotiqGrey">

Commit message: moveit config ok

File: ur10e_robotiq_simplified_description/urdf/ur10e_robotiq.urdf.xacro (robot description, xacro)
@@ -1,11 +1,10 @@
 <?xml version="1.0"?>
-<robot xmlns:xacro="http://ros.org/wiki/xacro"
-       name="ur10e_robotiq_simplified" >
+<robot xmlns:xacro="http://ros.org/wiki/xacro" name="ur10e_robotiq_simplified" >
   <!-- common stuff -->
-  <xacro:include filename="$(find ur_description)/urdf/inc/ur_common.xacro" />
+  <!-- <xacro:include filename="$(find ur_description)/urdf/inc/ur_common.xacro" /> -->
   <!-- ur10e -->
-  <xacro:include filename="$(find ur_simplified_description)/urdf/ur10e.urdf.xacro" />
-	<xacro:include filename="$(find ur10e_robotiq_simplified_description)/urdf/robotiq_arg2f_85_model_macro.xacro" />
+  <xacro:include filename="$(find ur_simplified_description)/urdf/ur10e/ur10e.xacro" />
   <!-- gripper -->
+  <xacro:include filename="$(find ur10e_robotiq_simplified_description)/urdf/robotiq_arg2f_85_model_macro.xacro" />
   <joint name="rq_coupler_joint" type="fixed">
     <parent link="tool0" />
@@ -37,5 +36,5 @@
   </inertial>
   </link>
-    <joint name="robotiq_joint" type="fixed">
+  <joint name="robotiq_joint" type="fixed">
     <parent link="robotiq_coupler" />
     <child link = "robotiq_arg2f_base_link" />
@@ -77,5 +76,5 @@
     </collision>
   </link>
-      <joint name="robotiq_joint_simplified" type="fixed">
+    <joint name="robotiq_joint_simplified" type="fixed">
       <parent link="robotiq_coupler" />
       <child link = "robotiq_simplified" />

File: ur10e_robotiq_simplified_description/urdf/ur10e_robotiq_robot.urdf.xacro (robot description, xacro)
@@ -4,14 +4,3 @@
   <!-- ur10e+robotiq -->
   <xacro:include filename="$(find ur10e_robotiq_simplified_description)/urdf/ur10e_robotiq.urdf.xacro" />
-  <!-- arm -->
-  <xacro:arg name="kinematics_config" default="$(find ur_description)/config/ur10e_default.yaml"/>
-  <xacro:ur10e_robot prefix="" joint_limited="false"
-    kinematics_file="${load_yaml('$(arg kinematics_config)')}"
-  />
-  <link name="world" />
-  <joint name="world_joint" type="fixed">
-    <parent link="world" />
-    <child link = "base_link" />
-    <origin xyz="0.0 0.0 0.0" rpy="0.0 0.0 0.0" />
-  </joint>
 </robot>

Commit message: fixes

File: ur10e_robotiq_simplified_description/urdf/ur10e_robotiq.urdf.xacro (robot description, xacro)
@@ -1,18 +1,26 @@
 <?xml version="1.0"?>
-<robot xmlns:xacro="http://ros.org/wiki/xacro"
-  name="ur10e_robotiq_simplified"
-  params=
-  "prefix
-  joint_limits_parameters_file
-  kinematics_parameters_file
-  physical_parameters_file
-  visual_parameters_file
-  transmission_hw_interface:=hardware_interface/PositionJointInterface
-  safety_limits:=false
-  safety_pos_margin:=0.15
-  safety_k_position:=20"
->
+<robot xmlns:xacro="http://ros.org/wiki/xacro" name="ur10e_robotiq_simplified">
+  <xacro:macro name="ur10e_robotiq_simplified" params=
+   "prefix:=''
+    joint_limits_parameters_file:='$(find ur_description)/config/ur10e/joint_limits.yaml'
+    kinematics_parameters_file:='$(find ur_description)/config/ur10e/default_kinematics.yaml'
+    physical_parameters_file:='$(find ur_description)/config/ur10e/physical_parameters.yaml'
+    transmission_hw_interface:=hardware_interface/PositionJointInterface
+    safety_limits:=false
+    safety_pos_margin:=0.15
+    safety_k_position:=20 ">
   <!-- ur10e -->
-  <xacro:include filename="$(find ur_description)/urdf/inc/ur10e_macro.xacro" />
+  <xacro:include filename="$(find ur_description)/urdf/inc/ur10e_macro.xacro"/>
+  <xacro:ur10e_robot
+    prefix = "${prefix}"
+    joint_limits_parameters_file="${joint_limits_parameters_file}"
+    kinematics_parameters_file="${kinematics_parameters_file}"
+    physical_parameters_file="${physical_parameters_file}"
+    visual_parameters_file='$(find ur_simplified_description)/config/ur10e/simplified_visual_parameters.yaml'
+    transmission_hw_interface="${transmission_hw_interface}"
+    safety_limits="${safety_limits}"
+    safety_pos_margin="${safety_pos_margin}"
+    safety_k_position="${safety_k_position}"
+  />
   <!-- gripper -->
   <xacro:include filename="$(find ur10e_robotiq_simplified_description)/urdf/robotiq_arg2f_85_model_macro.xacro" />
@@ -128,3 +136,4 @@
      </collision>
   </link>
+  </xacro:macro>
 </robot>

File: ur10e_robotiq_simplified_description/urdf/ur10e_robotiq_robot.urdf.xacro (robot description, xacro)
@@ -1,6 +1,6 @@
 <?xml version="1.0"?>
-<robot xmlns:xacro="http://ros.org/wiki/xacro"
-       name="ur10e_robotiq_simplified" >
+<robot xmlns:xacro="http://ros.org/wiki/xacro" name="ur10e_robotiq_simplified" >
   <!-- ur10e+robotiq -->
   <xacro:include filename="$(find ur10e_robotiq_simplified_description)/urdf/ur10e_robotiq.urdf.xacro" />
+  <xacro:ur10e_robotiq_simplified /> <!--DO NOT DELETE -->
 </robot>
