Commit message: remove robotiq

File: ur10e_robotiq_simplified_description/urdf/robotiq_arg2f_85_model_macro.xacro (robot description, xacro)
@@ -97,5 +97,5 @@
   </xacro:macro>
   <xacro:macro name="inner_knuckle_joint" params="prefix fingerprefix reflect">
-    <joint name="${prefix}${fingerprefix}_inner_knuckle_joint" type="revolute">
+    <joint name="${prefix}${fingerprefix}_inner_knuckle_joint" type="fixed">
       <!-- <origin xyz="0 ${reflect * -0.0127} 0.06142" rpy="${pi / 2 + .725} 0 ${(reflect - 1) * pi / 2}" /> -->
       <origin xyz="0 ${reflect * -0.0127} 0.06142" rpy="0 0 ${(1 + reflect) * pi / 2}"/>
@@ -108,5 +108,5 @@
   </xacro:macro>
   <xacro:macro name="inner_finger_joint" params="prefix fingerprefix">
-    <joint name="${prefix}${fingerprefix}_inner_finger_joint" type="revolute">
+    <joint name="${prefix}${fingerprefix}_inner_finger_joint" type="fixed">
       <origin xyz="0 0.0061 0.0471" rpy="0 0 0"/>
       <parent link="${prefix}${fingerprefix}_outer_finger" />
@@ -127,5 +127,5 @@
   <xacro:include filename="$(find ur10e_robotiq_simplified_description)/urdf/robotiq_arg2f.xacro" />
   <xacro:macro name="finger_joint" params="prefix">
-    <joint name="${prefix}finger_joint" type="revolute">
+    <joint name="${prefix}finger_joint" type="fixed">
       <origin xyz="0 -0.0306011 0.054904" rpy="0 0 ${pi}"/>
       <parent link="${prefix}robotiq_arg2f_base_link" />
@@ -137,5 +137,5 @@
   </xacro:macro>
   <xacro:macro name="right_outer_knuckle_joint" params="prefix">
-    <joint name="${prefix}right_outer_knuckle_joint" type="revolute">
+    <joint name="${prefix}right_outer_knuckle_joint" type="fixed">
       <origin xyz="0 0.0306011 0.054904" rpy="0 0 0"/>
       <parent link="${prefix}robotiq_arg2f_base_link" />

File: ur10e_robotiq_simplified_description/urdf/ur10e_robotiq.urdf.xacro (robot description, xacro)
@@ -37,4 +37,5 @@
   </inertial>
   </link>
+  <!--
     <joint name="robotiq_joint" type="fixed">
     <parent link="robotiq_coupler" />
@@ -42,5 +43,5 @@
     <origin xyz="0.0 0.0 0.0" rpy="0 0 ${0.0*pi}" />
   </joint>
-    <xacro:robotiq_arg2f_85 prefix=""/>
+    <xacro:robotiq_arg2f_85 prefix=""/>-->
   <link name="robotiq_simplified">
     <inertial>

Commit message: no collision robotiq

File: ur10e_robotiq_simplified_description/urdf/robotiq_arg2f_85_model_macro.xacro (robot description, xacro)
@@ -18,4 +18,7 @@
         </material>
       </visual>
+      <collision>
+            <!--   NO COLLISIONS  -->
+      </collision>
     </link>
   </xacro:macro>
@@ -36,4 +39,7 @@
         </material>
       </visual>
+      <collision>
+            <!--   NO COLLISIONS  -->
+      </collision>
     </link>
   </xacro:macro>
@@ -54,4 +60,7 @@
         </material>
       </visual>
+      <collision>
+            <!--   NO COLLISIONS  -->
+      </collision>
     </link>
   </xacro:macro>
@@ -72,4 +81,7 @@
         </material>
       </visual>
+      <collision>
+            <!--   NO COLLISIONS  -->
+      </collision>
     </link>
   </xacro:macro>
@@ -86,4 +98,7 @@
         </material>
       </visual>
+      <collision>
+            <!--   NO COLLISIONS  -->
+      </collision>
     </link>
   </xacro:macro>
