Commit message: fix

File: ur10e_robotiq_simplified_description/urdf/robotiq_arg2f.xacro (robot description, xacro)
@@ -3,9 +3,9 @@
   <xacro:macro name="robotiq_arg2f_base_link" params="prefix">
     <link name="${prefix}robotiq_arg2f_base_link">
-      <inertial>
+      <!-- <inertial>
         <origin xyz="8.625E-08 -4.6583E-06 0.03145" rpy="0 0 0" />
         <mass value="0.22652" />
         <inertia ixx="0.00020005" ixy="-4.2442E-10" ixz="-2.9069E-10" iyy="0.00017832" iyz="-3.4402E-08" izz="0.00013478" />
-      </inertial>
+      </inertial> -->
       <visual>
         <origin xyz="0 0 0" rpy="0 0 0" />
@@ -17,4 +17,9 @@
         </material>
       </visual>
+      <collision>
+        <geometry>
+            <cylinder length="0.0" radius="0.0"/>          <!--   NO COLLISIONS  -->
+        </geometry>
+      </collision>
     </link>
   </xacro:macro>

File: ur10e_robotiq_simplified_description/urdf/robotiq_arg2f_85_model_macro.xacro (robot description, xacro)
@@ -19,5 +19,7 @@
       </visual>
       <collision>
-            <!--   NO COLLISIONS  -->
+        <geometry>
+            <cylinder length="0.0" radius="0.0"/>          <!--   NO COLLISIONS  -->
+        </geometry>
       </collision>
     </link>
@@ -40,5 +42,7 @@
       </visual>
       <collision>
-            <!--   NO COLLISIONS  -->
+        <geometry>
+            <cylinder length="0.0" radius="0.0"/>          <!--   NO COLLISIONS  -->
+        </geometry>
       </collision>
     </link>
@@ -61,5 +65,7 @@
       </visual>
       <collision>
-            <!--   NO COLLISIONS  -->
+        <geometry>
+            <cylinder length="0.0" radius="0.0"/>          <!--   NO COLLISIONS  -->
+        </geometry>
       </collision>
     </link>
@@ -82,5 +88,7 @@
       </visual>
       <collision>
-            <!--   NO COLLISIONS  -->
+        <geometry>
+            <cylinder length="0.0" radius="0.0"/>          <!--   NO COLLISIONS  -->
+        </geometry>
       </collision>
     </link>
@@ -99,5 +107,7 @@
       </visual>
       <collision>
-            <!--   NO COLLISIONS  -->
+        <geometry>
+            <cylinder length="0.0" radius="0.0"/>          <!--   NO COLLISIONS  -->
+        </geometry>
       </collision>
     </link>

File: ur10e_robotiq_simplified_description/urdf/ur10e_robotiq.urdf.xacro (robot description, xacro)
@@ -37,10 +37,10 @@
   </inertial>
   </link>
-    <joint name="robotiq_joint" type="fixed">
+  <!-- <joint name="robotiq_joint" type="fixed">
     <parent link="robotiq_coupler" />
     <child link = "robotiq_arg2f_base_link" />
     <origin xyz="0.0 0.0 0.0" rpy="0 0 ${0.0*pi}" />
   </joint>
-    <xacro:robotiq_arg2f_85 prefix=""/>
+    <xacro:robotiq_arg2f_85 prefix=""/> -->
   <link name="robotiq_simplified">
     <inertial>

Commit message: no visual robotiq due to bugs

File: ur10e_robotiq_simplified_description/urdf/robotiq_arg2f.xacro (robot description, xacro)
@@ -17,4 +17,9 @@
         </material>
       </visual>
+      <collision>
+        <geometry>
+          <cylinder length="0.0" radius="0.0"/>          <!--   NO COLLISIONS  -->
+        </geometry>
+      </collision>
     </link>
   </xacro:macro>

File: ur10e_robotiq_simplified_description/urdf/robotiq_arg2f_85_model_macro.xacro (robot description, xacro)
@@ -18,4 +18,9 @@
         </material>
       </visual>
+      <collision>
+        <geometry>
+          <cylinder length="0.0" radius="0.0"/>          <!--   NO COLLISIONS  -->
+        </geometry>
+      </collision>
     </link>
   </xacro:macro>
@@ -36,4 +41,9 @@
         </material>
       </visual>
+      <collision>
+        <geometry>
+            <cylinder length="0.0" radius="0.0"/>          <!--   NO COLLISIONS  -->
+        </geometry>
+      </collision>
     </link>
   </xacro:macro>
@@ -54,4 +64,9 @@
         </material>
       </visual>
+      <collision>
+        <geometry>
+          <cylinder length="0.0" radius="0.0"/>          <!--   NO COLLISIONS  -->
+        </geometry>
+      </collision>
     </link>
   </xacro:macro>
@@ -72,4 +87,9 @@
         </material>
       </visual>
+      <collision>
+        <geometry>
+          <cylinder length="0.0" radius="0.0"/>          <!--   NO COLLISIONS  -->
+        </geometry>
+      </collision>
     </link>
   </xacro:macro>
@@ -86,4 +106,9 @@
         </material>
       </visual>
+      <collision>
+        <geometry>
+          <cylinder length="0.0" radius="0.0"/>          <!--   NO COLLISIONS  -->
+        </geometry>
+      </collision>
     </link>
   </xacro:macro>

File: ur10e_robotiq_simplified_description/urdf/ur10e_robotiq.urdf.xacro (robot description, xacro)
@@ -24,5 +24,5 @@
   />
   <!-- gripper -->
-  <xacro:include filename="$(find ur10e_robotiq_simplified_description)/urdf/robotiq_arg2f_85_model_macro.xacro" />
+  <!-- <xacro:include filename="$(find ur10e_robotiq_simplified_description)/urdf/robotiq_arg2f_85_model_macro.xacro" /> -->
   <joint name="rq_coupler_joint" type="fixed">
     <parent link="tool0" />
@@ -54,10 +54,10 @@
   </inertial>
   </link>
-  <joint name="robotiq_joint" type="fixed">
+  <!-- <joint name="robotiq_joint" type="fixed">
     <parent link="robotiq_coupler" />
     <child link = "robotiq_arg2f_base_link" />
     <origin xyz="0.0 0.0 0.0" rpy="0 0 ${0.0*pi}" />
   </joint>
-    <xacro:robotiq_arg2f_85 prefix=""/>
+    <xacro:robotiq_arg2f_85 prefix=""/> -->
   <link name="robotiq_simplified">
     <inertial>
