Commit message: fix robotiq visual

File: ur10e_robotiq_simplified_description/urdf/robotiq_arg2f_85_description.xacro (robot description, xacro)
@@ -2,5 +2,27 @@
 <robot xmlns:xacro="http://ros.org/wiki/xacro">
   <xacro:include filename="$(find robotiq_2f_85_gripper_visualization)/urdf/robotiq_arg2f_transmission.xacro" />
-  <xacro:include filename="$(find ur10e_robotiq_simplified_description)/urdf/robotiq_arg2f.xacro" />
+<xacro:macro name="robotiq_arg2f_base_link" params="prefix">
+    <link name="${prefix}robotiq_arg2f_base_link">
+      <!-- <inertial>
+        <origin xyz="8.625E-08 -4.6583E-06 0.03145" rpy="0 0 0" />
+        <mass value="0.22652" />
+        <inertia ixx="0.00020005" ixy="-4.2442E-10" ixz="-2.9069E-10" iyy="0.00017832" iyz="-3.4402E-08" izz="0.00013478" />
+      </inertial> -->
+      <visual>
+        <origin xyz="0 0 0" rpy="0 0 0" />
+        <geometry>
+          <mesh filename="package://robotiq_2f_85_gripper_visualization/meshes/visual/robotiq_arg2f_85_base_link.dae" scale="0.001 0.001 0.001"/>
+        </geometry>
+        <material name="">
+          <color rgba="0.1 0.1 0.1 1" />
+        </material>
+      </visual>
+      <collision>
+        <geometry>
+          <cylinder length="0.0" radius="0.0"/>          <!--   NO COLLISIONS  -->
+        </geometry>
+      </collision>
+    </link>
+  </xacro:macro>
   <xacro:macro name="outer_knuckle" params="prefix fingerprefix stroke">
     <link name="${prefix}${fingerprefix}_outer_knuckle">
@@ -172,4 +194,17 @@
     </joint>
     <xacro:finger_joints prefix="${prefix}" fingerprefix="right" reflect="-1.0"/>
+  </xacro:macro>
+  <xacro:macro name="finger_joints" params="prefix fingerprefix reflect">
+    <xacro:outer_finger_joint prefix="${prefix}" fingerprefix="${fingerprefix}"/>
+    <xacro:inner_knuckle_joint prefix="${prefix}" fingerprefix="${fingerprefix}" reflect="${reflect}"/>
+    <xacro:inner_finger_joint prefix="${prefix}" fingerprefix="${fingerprefix}"/>
+    <xacro:inner_finger_pad_joint prefix="${prefix}" fingerprefix="${fingerprefix}"/>
+  </xacro:macro>
+  <xacro:macro name="finger_links" params="prefix fingerprefix stroke">
+    <xacro:outer_knuckle prefix="${prefix}" fingerprefix="${fingerprefix}" stroke="${stroke}"/>
+    <xacro:outer_finger prefix="${prefix}" fingerprefix="${fingerprefix}" stroke="${stroke}"/>
+    <xacro:inner_finger prefix="${prefix}" fingerprefix="${fingerprefix}" stroke="${stroke}"/>
+    <xacro:inner_finger_pad prefix="${prefix}" fingerprefix="${fingerprefix}"/>
+    <xacro:inner_knuckle prefix="${prefix}" fingerprefix="${fingerprefix}" stroke="${stroke}"/>
   </xacro:macro>
   <!-- Initialization of all joints and links -->

File: ur10e_robotiq_simplified_description/urdf/ur10e_robotiq.urdf.xacro (robot description, xacro)
@@ -25,4 +25,5 @@
   <!-- gripper -->
   <!-- <xacro:include filename="$(find ur10e_robotiq_simplified_description)/urdf/robotiq_arg2f_85_model_macro.xacro" /> -->
+  <xacro:include filename="$(find ur10e_robotiq_simplified_description)/urdf/robotiq_arg2f_85_complete.xacro" />
   <!-- gripper -->
   <joint name="rq_coupler_joint" type="fixed">
@@ -55,10 +56,16 @@
   </inertial>
   </link>
-  <!-- <joint name="robotiq_joint" type="fixed">
+  <!-- <xacro:robotiq_arg2f_base_link prefix=""/>
+  <xacro:finger_joints prefix=""/>
+  <xacro:finger_links prefix=""/>
+  <xacro:finger_joints fingerprefix=""/>
+  <xacro:finger_joints reflect="1"/>
+  <xacro:finger_links fingerprefix=""/>
+  <xacro:finger_links stroke="0.05"/> -->
+  <joint name="robotiq_joint" type="fixed">
     <parent link="robotiq_coupler" />
     <child link = "robotiq_arg2f_base_link" />
     <origin xyz="0.0 0.0 0.0" rpy="0 0 ${0.0*pi}" />
   </joint>
-    <xacro:robotiq_arg2f_85 prefix=""/> -->
   <link name="robotiq_simplified">
     <inertial>
@@ -95,5 +102,5 @@
     </collision>
   </link>
-    <joint name="robotiq_joint_simplified" type="fixed">
+     <joint name="robotiq_joint_simplified" type="fixed">
       <parent link="robotiq_coupler" />
       <child link = "robotiq_simplified" />

Commit message: fix

File: ur10e_robotiq_simplified_description/urdf/robotiq_arg2f_85_description.xacro (robot description, xacro)
@@ -18,9 +18,9 @@
         </material>
       </visual>
-      <collision>
-        <geometry>
-          <cylinder length="0.0" radius="0.0"/>          <!--   NO COLLISIONS  -->
-        </geometry>
-      </collision>
+      <!-- <collision>
+        <geometry>
+          <cylinder length="0.0" radius="0.0"/>
+        </geometry>
+      </collision> -->
     </link>
   </xacro:macro>
@@ -41,10 +41,10 @@
         </material>
       </visual>
-      <collision>
-        <geometry>
-          <cylinder length="0.0" radius="0.0"/>          <!--   NO COLLISIONS  -->
-            <cylinder length="0.0" radius="0.0"/>          <!--   NO COLLISIONS  -->
-        </geometry>
-      </collision>
+      <!-- <collision>
+        <geometry>
+          <cylinder length="0.0" radius="0.0"/>
+            <cylinder length="0.0" radius="0.0"/>
+        </geometry>
+      </collision> -->
     </link>
   </xacro:macro>
@@ -65,9 +65,9 @@
         </material>
       </visual>
-      <collision>
-        <geometry>
-            <cylinder length="0.0" radius="0.0"/>          <!--   NO COLLISIONS  -->
-        </geometry>
-      </collision>
+      <!-- <collision>
+        <geometry>
+            <cylinder length="0.0" radius="0.0"/>
+        </geometry>
+      </collision> -->
     </link>
   </xacro:macro>
@@ -88,9 +88,9 @@
         </material>
       </visual>
-      <collision>
-        <geometry>
-          <cylinder length="0.0" radius="0.0"/>          <!--   NO COLLISIONS  -->
-        </geometry>
-      </collision>
+      <!-- <collision>
+        <geometry>
+          <cylinder length="0.0" radius="0.0"/>
+        </geometry>
+      </collision>  -->
     </link>
   </xacro:macro>
@@ -111,9 +111,9 @@
         </material>
       </visual>
-      <collision>
-        <geometry>
-          <cylinder length="0.0" radius="0.0"/>          <!--   NO COLLISIONS  -->
-        </geometry>
-      </collision>
+      <!-- <collision>
+        <geometry>
+          <cylinder length="0.0" radius="0.0"/>
+        </geometry>
+      </collision> -->
     </link>
   </xacro:macro>
@@ -130,9 +130,9 @@
         </material>
       </visual>
-      <collision>
-        <geometry>
-          <cylinder length="0.0" radius="0.0"/>          <!--   NO COLLISIONS  -->
-        </geometry>
-      </collision>
+      <!-- <collision>
+        <geometry>
+          <cylinder length="0.0" radius="0.0"/>
+        </geometry>
+      </collision> -->
     </link>
   </xacro:macro>
